File: LPC82x_ECG.kicad_pcb (KiCad board)
At the start: 2 copper layers, 4 parts, among them U1 ADS1292R, U2 LPC824

Commit message: no comment
Parts:
- moved R1 0.90 mm to (139.1, 113.7), turned to 90 degrees
Routing:
- net Net-(U1-Pad22): track 0.00 -> 6.21 mm
- net Net-(U1-Pad21): track 0.00 -> 6.15 mm
- net Net-(U1-Pad20): track 0.00 -> 6.09 mm
- net Net-(U1-Pad19): track 0.00 -> 6.02 mm
- net Net-(U1-Pad17): track 0.00 -> 5.46 mm
- net Net-(U1-Pad18): track 0.00 -> 5.40 mm
- net +3V3: track 0.00 -> 3.92 mm
- net GND: track 0.00 -> 3.58 mm
Other:
- board outline added: 25.4 x 17.8 mm
Changed lines of the file:
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@@
   (general
     (links 11)
-    (no_connects 11)
-    (area 0 0 0 0)
+    (no_connects 3)
+    (area 132.004999 98.984999 157.555001 116.915001)
     (thickness 1.6)
-    (drawings 0)
-    (tracks 0)
+    (drawings 4)
+    (tracks 23)
     (zones 0)
     (modules 4)
@@
   )
   (module Resistors_SMD:R_0603_HandSoldering (layer F.Cu)
-    (at 138.43 113.03)
+    (at 139.065 113.665 90)
     (descr "Resistor SMD 0603, hand soldering")
     (tags "resistor 0603")
     (attr smd)
-    (fp_text reference R1 (at 0 -1.45) (layer F.SilkS)
-      (effects (font (size 1 1) (thickness 0.15)))
-    )
-    (fp_text value R (at 0 1.55) (layer F.Fab)
-      (effects (font (size 1 1) (thickness 0.15)))
-    )
-    (fp_text user %R (at 0 0) (layer F.Fab)
+    (fp_text reference R1 (at 0 -1.45 90) (layer F.SilkS)
+      (effects (font (size 1 1) (thickness 0.15)))
+    )
+    (fp_text value R (at 0 1.55 90) (layer F.Fab)
+      (effects (font (size 1 1) (thickness 0.15)))
+    )
+    (fp_text user %R (at 0 0 90) (layer F.Fab)
       (effects (font (size 0.5 0.5) (thickness 0.075)))
     )
@@
     (fp_line (start 1.95 0.7) (end 1.95 -0.7) (layer F.CrtYd) (width 0.05))
     (fp_line (start 1.95 0.7) (end -1.96 0.7) (layer F.CrtYd) (width 0.05))
-    (pad 1 smd rect (at -1.1 0) (size 1.2 0.9) (layers F.Cu F.Paste F.Mask)
+    (pad 1 smd rect (at -1.1 0 90) (size 1.2 0.9) (layers F.Cu F.Paste F.Mask)
       (net 3 "Net-(R1-Pad1)"))
-    (pad 2 smd rect (at 1.1 0) (size 1.2 0.9) (layers F.Cu F.Paste F.Mask)
+    (pad 2 smd rect (at 1.1 0 90) (size 1.2 0.9) (layers F.Cu F.Paste F.Mask)
       (net 1 GND))
     (model ${KISYS3DMOD}/Resistors_SMD.3dshapes/R_0603.wrl
@@
     )
   )
+  (gr_line (start 132.08 116.84) (end 132.08 99.06) (angle 90) (layer Edge.Cuts) (width 0.15))
+  (gr_line (start 157.48 116.84) (end 132.08 116.84) (angle 90) (layer Edge.Cuts) (width 0.15))
+  (gr_line (start 157.48 99.06) (end 157.48 116.84) (angle 90) (layer Edge.Cuts) (width 0.15))
+  (gr_line (start 132.08 99.06) (end 157.48 99.06) (angle 90) (layer Edge.Cuts) (width 0.15))
+  (segment (start 151.4511 104.6786) (end 154.7214 104.6786) (width 0.25) (layer F.Cu) (net 1))
+  (segment (start 154.7214 104.6786) (end 154.94 104.46) (width 0.25) (layer F.Cu) (net 1))
+  (segment (start 151.4511 105.3286) (end 153.9086 105.3286) (width 0.25) (layer F.Cu) (net 2))
+  (segment (start 153.9086 105.3286) (end 154.94 106.36) (width 0.25) (layer F.Cu) (net 2))
+  (segment (start 140.41 107.16) (end 142.36 107.16) (width 0.25) (layer F.Cu) (net 19))
+  (segment (start 143.1286 107.9286) (end 145.5511 107.9286) (width 0.25) (layer F.Cu) (net 19))
+  (segment (start 142.36 107.16) (end 143.1286 107.9286) (width 0.25) (layer F.Cu) (net 19))
+  (segment (start 140.41 106.66) (end 142.66 106.66) (width 0.25) (layer F.Cu) (net 20))
+  (segment (start 143.2786 107.2786) (end 145.5511 107.2786) (width 0.25) (layer F.Cu) (net 20))
+  (segment (start 142.66 106.66) (end 143.2786 107.2786) (width 0.25) (layer F.Cu) (net 20))
+  (segment (start 140.41 106.16) (end 142.44 106.16) (width 0.25) (layer F.Cu) (net 21))
+  (segment (start 144.5714 104.0286) (end 145.5511 104.0286) (width 0.25) (layer F.Cu) (net 21))
+  (segment (start 142.44 106.16) (end 144.5714 104.0286) (width 0.25) (layer F.Cu) (net 21))
+  (segment (start 140.41 105.66) (end 142.24 105.66) (width 0.25) (layer F.Cu) (net 22))
+  (segment (start 144.5 103.4) (end 145.5297 103.4) (width 0.25) (layer F.Cu) (net 22))
+  (segment (start 142.24 105.66) (end 144.5 103.4) (width 0.25) (layer F.Cu) (net 22))
+  (segment (start 145.5297 103.4) (end 145.5511 103.3786) (width 0.25) (layer F.Cu) (net 22))
+  (segment (start 140.41 105.16) (end 141.94 105.16) (width 0.25) (layer F.Cu) (net 23))
+  (segment (start 144.3714 102.7286) (end 145.5511 102.7286) (width 0.25) (layer F.Cu) (net 23))
+  (segment (start 141.94 105.16) (end 144.3714 102.7286) (width 0.25) (layer F.Cu) (net 23))
+  (segment (start 140.41 104.66) (end 141.72 104.66) (width 0.25) (layer F.Cu) (net 24))
+  (segment (start 144.3014 102.0786) (end 145.5511 102.0786) (width 0.25) (layer F.Cu) (net 24))
+  (segment (start 141.72 104.66) (end 144.3014 102.0786) (width 0.25) (layer F.Cu) (net 24))
 )
